File: CO2-sensor.kicad_sch (KiCad schematic)
At the start: 41 parts, among them IC1 SCD41-D-R1, IC2 NCP1117ST33T3G, IC3 W25Q32JVSSIQ, J1 1734028-1, U1 RP2040, Y1 ABM8-272-T3

Commit message: yep
Parts:
- IC1: value SCD41-D-R1 -> a
Changed lines of the file:
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@@
 			)
 		)
-		(property "Value" "SCD41-D-R1"
+		(property "Value" "a"
 			(at 172.466 75.184 90)
 			(effects
